Commit message: added function set_gripper_position

File: robotiq_2f_model/model/robotiq_2f_85.urdf.xacro (robot description, xacro)
@@ -21,12 +21,12 @@
 </xacro:macro -->
 <robot xmlns:xacro="http://ros.org/wiki/xacro">
-	<xacro:macro name="robotiq_2f_85" params="parent name precise_collision:=false adaptive_transmission:=false with_pads:=true *origin">
+	<xacro:macro name="robotiq_2f_85" params="parent joint_name name precise_collision:=false adaptive_transmission:=false with_pads:=true *origin">
 		<!-- base -->
-		<joint name="${parent}_${name}_base_joint" type="fixed">
+		<joint name="${parent}_${name}_BASE_joint" type="fixed">
 			<xacro:insert_block name="origin"/>
 			<parent link="${parent}"/>
-			<child link="${name}_base"/>
-		</joint>
-		<link name="${name}_base">
+			<child link="${name}_BASE"/>
+		</joint>
+		<link name="${name}_BASE">
 			<!-- inertial>
 				<mass value="0.1"/>
@@ -62,7 +62,7 @@
 		</link>
 		<!-- right finger -->
-		<joint name="${name}_right_driver_joint" type="revolute">
+		<joint name="${joint_name}" type="revolute">
 			<origin xyz="0 0.0306011 0.054904" rpy="0 0 0"/>
-			<parent link="${name}_base"/>
+			<parent link="${name}_BASE"/>
 			<child link="${name}_right_driver"/>
 			<axis xyz="1 0 0"/>
@@ -146,5 +146,5 @@
 			<limit lower="${-170 * 3.141592 / 180}" upper="${170 * 3.141592 / 180}" effort="176" velocity="${110 * 3.141592 / 180}" />
 			<xacro:unless value="${adaptive_transmission}">
-			<mimic joint="${name}_right_driver_joint" multiplier="-1"/>
+			<mimic joint="${joint_name}" multiplier="-1"/>
 			</xacro:unless>
 		</joint>
@@ -204,10 +204,10 @@
 		<joint name="${name}_right_spring_link_joint" type="revolute">
 			<origin xyz="0 0.012 0.0614" rpy="0 0 0"/>
-			<parent link="${name}_base"/>
+			<parent link="${name}_BASE"/>
 			<child link="${name}_right_spring_link"/>
 			<axis xyz="1 0 0"/>
 			<limit lower="${-170 * 3.141592 / 180}" upper="${170 * 3.141592 / 180}" effort="176" velocity="${110 * 3.141592 / 180}" />
 			<xacro:unless value="${adaptive_transmission}">
-			<mimic joint="${name}_right_driver_joint" multiplier="1"/>
+			<mimic joint="${joint_name}" multiplier="1"/>
 			</xacro:unless>
 		</joint>
@@ -242,10 +242,10 @@
 		<joint name="${name}_left_driver_joint" type="revolute">
 			<origin xyz="0 -0.0306011 0.054904" rpy="0 0 3.141592653589793"/>
-			<parent link="${name}_base"/>
+			<parent link="${name}_BASE"/>
 			<child link="${name}_left_driver"/>
 			<axis xyz="1 0 0"/>
 			<limit lower="${0 * 3.141592 / 180}" upper="${41 * 3.141592 / 180}" effort="176" velocity="${110 * 3.141592 / 180}" />
 			<xacro:unless value="${adaptive_transmission}">
-			<mimic joint="${name}_right_driver_joint" multiplier="1"/>
+			<mimic joint="${joint_name}" multiplier="1"/>
 			</xacro:unless>
 		</joint>
@@ -327,5 +327,5 @@
 			<limit lower="${-170 * 3.141592 / 180}" upper="${170 * 3.141592 / 180}" effort="176" velocity="${110 * 3.141592 / 180}" />
 			<xacro:unless value="${adaptive_transmission}">
-			<mimic joint="${name}_right_driver_joint" multiplier="-1"/>
+			<mimic joint="${joint_name}" multiplier="-1"/>
 			</xacro:unless>
 		</joint>
@@ -385,10 +385,10 @@
 		<joint name="${name}_left_spring_link_joint" type="revolute">
 			<origin xyz="0 -0.012 0.0614" rpy="0 0 3.141592653589793"/>
-			<parent link="${name}_base"/>
+			<parent link="${name}_BASE"/>
 			<child link="${name}_left_spring_link"/>
 			<axis xyz="1 0 0"/>
 			<limit lower="${-170 * 3.141592 / 180}" upper="${170 * 3.141592 / 180}" effort="176" velocity="${110 * 3.141592 / 180}" />
 			<xacro:unless value="${adaptive_transmission}">
-			<mimic joint="${name}_right_driver_joint" multiplier="1"/>
+			<mimic joint="${joint_name}" multiplier="1"/>
 			</xacro:unless>
 		</joint>
@@ -422,5 +422,5 @@
 		<transmission name="${name}_right_driver_trans">
 			<type>transmission_interface/SimpleTransmission</type>
-			<joint name="${name}_right_driver_joint">
+			<joint name="${joint_name}">
 				<hardwareInterface>hardware_interface/PositionJointInterface</hardwareInterface>
 			</joint>

Commit message: Added mimic joint plugins

File: robotiq_2f_model/model/robotiq_2f_85.urdf.xacro (robot description, xacro)
@@ -16,9 +16,6 @@
 	material properties, and simulation parameters.
 -->
-<!-- length is along the z-axis! -->
-<!-- xacro:macro name="cylinder_inertia" params="radius length mass">
-	<inertia ixx="${mass * (3 * radius * radius + length * length) / 12}" iyy="${mass * radius* radius / 2}" izz="${mass * (3 * radius * radius + length * length) / 12}" ixy="0" iyz="0" ixz="0"/>
-</xacro:macro -->
 <robot xmlns:xacro="http://ros.org/wiki/xacro">
+	<xacro:include filename="$(find robotiq_2f_model)/model/inertias.urdf.xacro" />
 	<xacro:macro name="robotiq_2f_85" params="parent joint_name name precise_collision:=false adaptive_transmission:=false with_pads:=true *origin">
 		<!-- base -->
@@ -29,12 +26,12 @@
 		</joint>
 		<link name="${name}_BASE">
-			<!-- inertial>
-				<mass value="0.1"/>
-				<origin xyz="0 0 0.055"  />
-				<cylinder_inertia radius="0.06" length="0.11" mass="0.1"/>
-			</inertial -->
-			<visual>
-				<geometry>
-					<mesh filename="package://robotiq_2f_model/model/meshes/2f85/visual/base.dae" scale="0.001 0.001 0.001"/>
+			<inertial>
+				<mass value="0.2"/>
+				<origin xyz="0 0 ${0.015*0.5}"  />
+				<cylinder_inertia radius="0.04" length="0.045" mass="0.2"/>
+			</inertial>
+			<visual>
+				<geometry>
+					<mesh filename="package://robotiq_2f_model/model/meshes/2f85/collision/base.stl" scale="0.001 0.001 0.001"/>
 				</geometry>
 			</visual>
@@ -70,9 +67,9 @@
 		</joint>
 		<link name="${name}_right_driver">
-			<!-- inertial>
-				<mass value="0.1"/>
-				<origin xyz="0 0 0.055"  />
-				<cylinder_inertia radius="0.06" length="0.11" mass="0.1"/>
-			</inertial -->
+			<inertial>
+				<mass value="0.05"/>
+				<origin xyz="0 0.02 0" rpy="0 0 0" />
+				<box_inertia x_dim="0.02" y_dim="0.04" z_dim="0.02" mass="0.05"/>
+			</inertial>
 			<visual>
 				<geometry>
@@ -113,9 +110,9 @@
 		</xacro:if>
 		<link name="${name}_right_coupler">
-			<!-- inertial>
-				<mass value="0.1"/>
-				<origin xyz="0 0 0.055"  />
-				<cylinder_inertia radius="0.06" length="0.11" mass="0.1"/>
-			</inertial -->
+			<inertial>
+				<mass value="0.05"/>
+				<origin xyz="0 0.0 0.025" rpy="-1.7 0 0"/>
+				<box_inertia x_dim="0.03" y_dim="0.065" z_dim="0.02" mass="0.05"/>
+			</inertial>
 			<visual>
 				<geometry>
@@ -150,4 +147,9 @@
 		</joint>
 		<link name="${name}_right_follower">
+			<inertial>
+				<mass value="0.05"/>
+				<origin xyz="0 -0.018 0.022" />
+				<box_inertia x_dim="0.02" y_dim="0.015" z_dim="0.048" mass="0.05"/>
+			</inertial>
 			<visual>
 				<geometry>
@@ -171,35 +173,37 @@
 			</xacro:if>
 		</link>
-		<joint name="${name}_right_pad_joint" type="fixed">
-			<parent link="${name}_right_follower"/>
-			<child link="${name}_right_pad"/>
-		</joint>
-		<link name="${name}_right_pad">
-			<!-- inertial>
-				<mass value="0.1"/>
-				<origin xyz="0 0 0.055"  />
-				<cylinder_inertia radius="0.06" length="0.11" mass="0.1"/>
-			</inertial -->
-			<visual>
-				<geometry>
-					<mesh filename="package://robotiq_2f_model/model/meshes/2f85/visual/pad.dae" scale="0.001 0.001 0.001"/>
-				</geometry>
-			</visual>
-			<xacro:unless value="${precise_collision}">
-			<collision>
-				<origin xyz="0 -0.022 0.031" rpy="0 0 0"/>
-				<geometry>
-					<box size="0.02 0.008 0.036"/>
-				</geometry>
-			</collision>
-			</xacro:unless>
-			<xacro:if value="${precise_collision}">
-			<collision>
-				<geometry>
-					<mesh filename="package://robotiq_2f_model/model/meshes/2f85/collision/pad.stl" scale="0.001 0.001 0.001"/>
-				</geometry>
-			</collision>
-			</xacro:if>
-		</link>
+		<xacro:if value="${with_pads}">
+			<joint name="${name}_right_pad_joint" type="fixed">
+				<parent link="${name}_right_follower"/>
+				<child link="${name}_right_pad"/>
+			</joint>
+			<link name="${name}_right_pad">
+				<inertial>
+					<mass value="0.01"/>
+					<origin xyz="0 -0.022 0.031" />
+					<box_inertia x_dim="0.02" y_dim="0.008" z_dim="0.036" mass="0.01"/>
+				</inertial>
+				<visual>
+					<geometry>
+						<mesh filename="package://robotiq_2f_model/model/meshes/2f85/visual/pad.dae" scale="0.001 0.001 0.001"/>
+					</geometry>
+				</visual>
+				<xacro:unless value="${precise_collision}">
+				<collision>
+					<origin xyz="0 -0.022 0.031" rpy="0 0 0"/>
+					<geometry>
+						<box size="0.02 0.008 0.036"/>
+					</geometry>
+				</collision>
+				</xacro:unless>
+				<xacro:if value="${precise_collision}">
+				<collision>
+					<geometry>
+						<mesh filename="package://robotiq_2f_model/model/meshes/2f85/collision/pad.stl" scale="0.001 0.001 0.001"/>
+					</geometry>
+				</collision>
+				</xacro:if>
+			</link>
+		</xacro:if>
 		<joint name="${name}_right_spring_link_joint" type="revolute">
 			<origin xyz="0 0.012 0.0614" rpy="0 0 0"/>
@@ -213,9 +217,9 @@
 		</joint>
 		<link name="${name}_right_spring_link">
-			<!-- inertial>
-				<mass value="0.1"/>
-				<origin xyz="0 0 0.055"  />
-				<cylinder_inertia radius="0.06" length="0.11" mass="0.1"/>
-			</inertial -->
+			<inertial>
+				<mass value="0.05"/>
+				<origin xyz="0 0.018 0.018" rpy="-0.7068 0 0"/>
+				<box_inertia x_dim="0.04" y_dim="0.02" z_dim="0.065" mass="0.05"/>
+			</inertial>
 			<visual>
 				<geometry>
@@ -245,5 +249,5 @@
 			<child link="${name}_left_driver"/>
 			<axis xyz="1 0 0"/>
-			<limit lower="${0 * 3.141592 / 180}" upper="${41 * 3.141592 / 180}" effort="176" velocity="${110 * 3.141592 / 180}" />
+			<limit lower="${0 * 3.141592 / 180}" upper="${50 * 3.141592 / 180}" effort="176" velocity="${110 * 3.141592 / 180}" />
 			<xacro:unless value="${adaptive_transmission}">
 			<mimic joint="${joint_name}" multiplier="1"/>
@@ -251,9 +255,9 @@
 		</joint>
 		<link name="${name}_left_driver">
-			<!-- inertial>
-				<mass value="0.1"/>
-				<origin xyz="0 0 0.055"  />
-				<cylinder_inertia radius="0.06" length="0.11" mass="0.1"/>
-			</inertial -->
+			<inertial>
+				<mass value="0.05"/>
+				<origin xyz="0 0.02 0" rpy="0 0 0" />
+				<box_inertia x_dim="0.02" y_dim="0.04" z_dim="0.02" mass="0.05"/>
+			</inertial>
 			<visual>
 				<geometry>
@@ -294,9 +298,9 @@
 		</xacro:if>
 		<link name="${name}_left_coupler">
-			<!-- inertial>
-				<mass value="0.1"/>
-				<origin xyz="0 0 0.055"  />
-				<cylinder_inertia radius="0.06" length="0.11" mass="0.1"/>
-			</inertial -->
+			<inertial>
+				<mass value="0.05"/>
+				<origin xyz="0 0.0 0.025" rpy="-1.7 0 0"/>
+				<box_inertia x_dim="0.03" y_dim="0.065" z_dim="0.02" mass="0.05"/>
+			</inertial>
 			<visual>
 				<geometry>
@@ -331,4 +335,9 @@
 		</joint>
 		<link name="${name}_left_follower">
+			<inertial>
+				<mass value="0.05"/>
+				<origin xyz="0 -0.018 0.022" />
+				<box_inertia x_dim="0.02" y_dim="0.015" z_dim="0.048" mass="0.05"/>
+			</inertial>
 			<visual>
 				<geometry>
@@ -352,35 +361,37 @@
 			</xacro:if>
 		</link>
-		<joint name="${name}_left_pad_joint" type="fixed">
-			<parent link="${name}_left_follower"/>
-			<child link="${name}_left_pad"/>
-		</joint>
-		<link name="${name}_left_pad">
-			<!-- inertial>
-				<mass value="0.1"/>
-				<origin xyz="0 0 0.055"  />
-				<cylinder_inertia radius="0.06" length="0.11" mass="0.1"/>
-			</inertial -->
-			<visual>
-				<geometry>
-					<mesh filename="package://robotiq_2f_model/model/meshes/2f85/visual/pad.dae" scale="0.001 0.001 0.001"/>
-				</geometry>
-			</visual>
-			<xacro:unless value="${precise_collision}">
-			<collision>
-				<origin xyz="0 -0.022 0.031" rpy="0 0 0"/>
-				<geometry>
-					<box size="0.02 0.008 0.036"/>
-				</geometry>
-			</collision>
-			</xacro:unless>
-			<xacro:if value="${precise_collision}">
-			<collision>
-				<geometry>
-					<mesh filename="package://robotiq_2f_model/model/meshes/2f85/collision/pad.stl" scale="0.001 0.001 0.001"/>
-				</geometry>
-			</collision>
-			</xacro:if>
-		</link>
+		<xacro:if value="${with_pads}">
+			<joint name="${name}_left_pad_joint" type="fixed">
+				<parent link="${name}_left_follower"/>
+				<child link="${name}_left_pad"/>
+			</joint>
+			<link name="${name}_left_pad">
+				<inertial>
+					<mass value="0.01"/>
+					<origin xyz="0 -0.022 0.031" />
+					<box_inertia x_dim="0.02" y_dim="0.008" z_dim="0.036" mass="0.01"/>
+				</inertial>
+				<visual>
+					<geometry>
+						<mesh filename="package://robotiq_2f_model/model/meshes/2f85/visual/pad.dae" scale="0.001 0.001 0.001"/>
+					</geometry>
+				</visual>
+				<xacro:unless value="${precise_collision}">
+				<collision>
+					<origin xyz="0 -0.022 0.031" rpy="0 0 0"/>
+					<geometry>
+						<box size="0.02 0.008 0.036"/>
+					</geometry>
+				</collision>
+				</xacro:unless>
+				<xacro:if value="${precise_collision}">
+				<collision>
+					<geometry>
+						<mesh filename="package://robotiq_2f_model/model/meshes/2f85/collision/pad.stl" scale="0.001 0.001 0.001"/>
+					</geometry>
+				</collision>
+				</xacro:if>
+			</link>
+		</xacro:if>
 		<joint name="${name}_left_spring_link_joint" type="revolute">
 			<origin xyz="0 -0.012 0.0614" rpy="0 0 3.141592653589793"/>
@@ -394,9 +405,9 @@
 		</joint>
 		<link name="${name}_left_spring_link">
-			<!-- inertial>
-				<mass value="0.1"/>
-				<origin xyz="0 0 0.055"  />
-				<cylinder_inertia radius="0.06" length="0.11" mass="0.1"/>
-			</inertial -->
+			<inertial>
+				<mass value="0.05"/>
+				<origin xyz="0 0.018 0.018" rpy="-0.7068 0 0"/>
+				<box_inertia x_dim="0.04" y_dim="0.02" z_dim="0.065" mass="0.05"/>
+			</inertial>
 			<visual>
 				<geometry>
@@ -420,13 +431,47 @@
 			</xacro:if>
 		</link>
-		<transmission name="${name}_right_driver_trans">
-			<type>transmission_interface/SimpleTransmission</type>
-			<joint name="${joint_name}">
-				<hardwareInterface>hardware_interface/PositionJointInterface</hardwareInterface>
-			</joint>
-			<actuator name="${name}_right_driver_motor">
-				<mechanicalReduction>1</mechanicalReduction>
-			</actuator>
-		</transmission>
+		<xacro:unless value="${adaptive_transmission}">
+			<transmission name="${name}_right_driver_trans">
+				<type>transmission_interface/SimpleTransmission</type>
+				<joint name="${joint_name}">
+					<hardwareInterface>hardware_interface/PositionJointInterface</hardwareInterface>
+				</joint>
+				<actuator name="${name}_right_driver_motor">
+					<mechanicalReduction>1</mechanicalReduction>
+				</actuator>
+			</transmission>
+			<gazebo>
+				<plugin name="${name}_right_follower_joint_plugin" filename="libroboticsgroup_gazebo_mimic_joint_plugin.so">
+					<joint>${joint_name}</joint>
+					<mimicJoint>${name}_right_follower_joint</mimicJoint>
+					<hasPID />
+					<multiplier>-1</multiplier>
+				</plugin>
+				<plugin name="${name}_right_spring_link_joint_plugin" filename="libroboticsgroup_gazebo_mimic_joint_plugin.so">
+					<joint>${joint_name}</joint>
+					<mimicJoint>${name}_right_spring_link_joint</mimicJoint>
+					<hasPID />
+					<multiplier>1</multiplier>
+				</plugin>
+				<plugin name="${name}_left_follower_joint_plugin" filename="libroboticsgroup_gazebo_mimic_joint_plugin.so">
+					<joint>${joint_name}</joint>
+					<mimicJoint>${name}_left_follower_joint</mimicJoint>
+					<hasPID />
+					<multiplier>-1</multiplier>
+				</plugin>
+				<plugin name="${name}_left_spring_link_joint_plugin" filename="libroboticsgroup_gazebo_mimic_joint_plugin.so">
+					<joint>${joint_name}</joint>
+					<mimicJoint>${name}_left_spring_link_joint</mimicJoint>
+					<hasPID />
+					<multiplier>1</multiplier>
+				</plugin>
+				<plugin name="${name}_left_driver_joint_plugin" filename="libroboticsgroup_gazebo_mimic_joint_plugin.so">
+					<joint>${joint_name}</joint>
+					<mimicJoint>${name}_left_driver_joint</mimicJoint>
+					<hasPID />
+					<multiplier>1</multiplier>
+				</plugin>
+			</gazebo>
+		</xacro:unless>
 	</xacro:macro>
 </robot>

Commit message: Added gazebo properties to model

File: robotiq_2f_model/model/robotiq_2f_85.urdf.xacro (robot description, xacro)
@@ -19,4 +19,15 @@
 	<xacro:include filename="$(find robotiq_2f_model)/model/inertias.urdf.xacro" />
 	<xacro:macro name="robotiq_2f_85" params="parent joint_name name precise_collision:=false adaptive_transmission:=false with_pads:=true *origin">
+                <xacro:property name="gripper_kp" value="1000000.0" />
+  		<xacro:property name="gripper_kd" value="1.5" />
+  		<xacro:property name="gripper_mu" value="1.2" />
+                <xacro:macro name="gazebo_params_gripper" params="name kp kd mu">
+    			<gazebo reference="${name}">
+      			<kp>${kp}</kp>
+      			<kd>${kd}</kd>
+      			<mu1>${mu}</mu1>
+      			<mu2>${mu}</mu2>
+    			</gazebo>
+  		</xacro:macro>
 		<!-- base -->
 		<joint name="${parent}_${name}_BASE_joint" type="fixed">
@@ -58,4 +69,5 @@
 			</xacro:if>
 		</link>
+		<xacro:gazebo_params_gripper name="${name}_BASE" kp ="${gripper_kp}" kd="${gripper_kd}" mu="${gripper_mu}"/>
 		<!-- right finger -->
 		<joint name="${joint_name}" type="revolute">
@@ -205,4 +217,5 @@
 				</xacro:if>
 			</link>
+			<xacro:gazebo_params_gripper name="${name}_right_pad" kp ="${gripper_kp}" kd="${gripper_kd}" mu="${gripper_mu}"/>
 		</xacro:if>
 		<joint name="${name}_right_spring_link_joint" type="revolute">
@@ -393,4 +406,5 @@
 				</xacro:if>
 			</link>
+			<xacro:gazebo_params_gripper name="${name}_left_pad" kp ="${gripper_kp}" kd="${gripper_kd}" mu="${gripper_mu}"/>
 		</xacro:if>
 		<joint name="${name}_left_spring_link_joint" type="revolute">

File: robotiq_2f_robot/robot/simple_rq2f85.urdf.xacro (robot description, xacro)
@@ -3,5 +3,5 @@
 	<xacro:include filename="$(find robotiq_2f_model)/model/robotiq_2f_85.urdf.xacro" />
 	<link name="world"/>
-	<xacro:robotiq_2f_85 name="simple_gripper" parent="world" precise_collision="false" adaptive_transmission="false">
+	<xacro:robotiq_2f_85 name="simple_gripper" joint_name="GRIPPER_JOINT" parent="world" precise_collision="false" adaptive_transmission="false">
 		<origin xyz="0 0 0" rpy="0 0 0"/>
 	</xacro:robotiq_2f_85>
